Commit message: Update panda camera, gripper controller, and MoveIt integration

File: src/panda/urdf/panda.xacro.urdf (robot description, URDF)
Before this commit: robot panda, 15 links, 14 joints
Links:
- added link panda_wrist_eye_marker_link, mass 0.001; visual box size=0.05 0.03 0.03
Joints:
- added joint panda_wrist_eye_marker_joint: type fixed, parent panda_link8, child panda_wrist_eye_marker_link, origin xyz=0.065 0 0.0 rpy=0 -1.5707963267948966 0
- joint panda_finger_joint2: mimic (none) -> joint=panda_finger_joint1
- joint panda_wrist_eye_joint: origin xyz=0 0 0.12 rpy=0 1.5707963267948966 0 -> xyz=0.065 0 0.0 rpy=0 -1.5707963267948966 0

Commit message: Revert "Standardize Panda MoveIt groups, gripper execution, and docs"
This reverts commit 3bc5807e2596c7dee3ec51c77211af92b7998d82.

File: src/panda/urdf/panda.xacro.urdf (robot description, URDF)
Before this commit: robot panda, 16 links, 15 joints
Joints:
- joint panda_finger_joint2: mimic (none) -> joint=panda_finger_joint1

Commit message: Working arm movement to pose.

File: src/panda/urdf/panda.xacro.urdf (robot description, URDF)
Before this commit: robot panda, 16 links, 15 joints
Links:
- removed link panda_wrist_eye_link
- added link panda_wrist_eye_sensor, mass 0.05; collision box size=0.03 0.02 0.02; visual box size=0.03 0.02 0.02
Joints:
- joint panda_wrist_eye_joint: child panda_wrist_eye_link -> panda_wrist_eye_sensor

Commit message: Optical frame added into urdf.  Working pick and place

File: src/panda/urdf/panda.xacro.urdf (robot description, URDF)
Before this commit: robot panda, 16 links, 15 joints
Links:
- added link panda_wrist_eye_optical_frame
Joints:
- added joint panda_wrist_eye_optical_joint: type fixed, parent panda_wrist_eye_sensor, child panda_wrist_eye_optical_frame, origin xyz=0 0 0 rpy=-1.5707963267948966 0 -1.5707963267948966
