Commit message: Add advance urdf concept files

File: src/robotic_arm_description/urdf/demo/demo_links.urdf (robot description, URDF)
Before this commit: robot demo_links, 2 links, 1 joints
Links:
- link base_link: geometry visual cylinder length=0.5 radius=0.2
Joints:
- joint base_link_to_link_1: axis (none) -> 0 0 1; limit (none) -> lower=-10.0 upper=10.0 effort=1000.0 velocity=0.5; origin xyz=0 0.3 0.0 -> xyz=0 0.0 0.0; type fixed -> revolute
